File: mtfjis.kicad_pcb (KiCad board)
At the start: 2 copper layers, 500 x 194 mm, 198 parts, among them J1 CONN_CAP_IBM_F

Commit message: gitignore mtfjis-backups, wipe tracks and update schematic
Parts:
- removed COL_1_TP9: C1_TestPoint, TestPoint:TestPoint_Pad_D1.0mm
- removed COL_2_TP10: C2_TestPoint, TestPoint:TestPoint_Pad_D1.0mm
- removed COL_3_TP11: C3_TestPoint, TestPoint:TestPoint_Pad_D1.0mm
- removed COL_4_TP12: C4_TestPoint, TestPoint:TestPoint_Pad_D1.0mm
- removed COL_5_TP13: C5_TestPoint, TestPoint:TestPoint_Pad_D1.0mm
- removed COL_6_TP14: C6_TestPoint, TestPoint:TestPoint_Pad_D1.0mm
- removed COL_7_TP15: C7_TestPoint, TestPoint:TestPoint_Pad_D1.0mm
- removed COL_8_TP16: C8_TestPoint, TestPoint:TestPoint_Pad_D1.0mm
- removed COL_9_TP17: C9_TestPoint, TestPoint:TestPoint_Pad_D1.0mm
- removed COL_A_TP18: CA_TestPoint, TestPoint:TestPoint_Pad_D1.0mm
- removed COL_B_TP19: CB_TestPoint, TestPoint:TestPoint_Pad_D1.0mm
- removed COL_C_TP20: CC_TestPoint, TestPoint:TestPoint_Pad_D1.0mm
- removed COL_D_TP21: CD_TestPoint, TestPoint:TestPoint_Pad_D1.0mm
- removed COL_E_TP22: CE_TestPoint, TestPoint:TestPoint_Pad_D1.0mm
- removed COL_F_TP23: CF_TestPoint, TestPoint:TestPoint_Pad_D1.0mm
- removed COL_G_TP24: CG_TestPoint, TestPoint:TestPoint_Pad_D1.0mm
- removed the SW_3_0 at (169.3, 201.8)
- removed SW_CENTER_0: D,3, lib_fp:SW_CAP_IBM_F_ALT
- added SW_JIS4_0: C7_R1, lib_fp:SW_CAP_IBM_F_ALT, F.Cu at (270.0, 355.6)
- added SW_LALT_0: C2_R1, lib_fp:SW_CAP_IBM_F_ALT, F.Cu at (341.1, 351.3)
- added SW_PAUS_0: CC_R8, lib_fp:SW_CAP_IBM_F_ALT, F.Cu at (357.4, 351.3)
- added SW_PRSC_0: CB_R8, lib_fp:SW_CAP_IBM_F_ALT, F.Cu at (341.1, 367.4)
- added SW_SCLK_0: CB_R7, lib_fp:SW_CAP_IBM_F, F.Cu at (357.4, 367.4)
- SWSW_NUMENT1: value G,2 -> CE_R4
- SW_0_0: value 9,5 -> C8_R7
- SW_2_0: renamed from SW_1_0; value 3,6 -> C2_R7
- SW_3_0: renamed from SW_2_0; value 4,6 -> C3_R7
- SW_4_0: value 5,5 -> C3_R6
- SW_5_0: value 6,6 -> C4_R7
- SW_6_0: value 7,6 -> C5_R7
- SW_7_0: value 8,5 -> C5_R6
- SW_8_0: value 8,6 -> C6_R7
- SW_9_0: value 9,6 -> C7_R6
- SW_APOS_0: value B,3 -> C9_R4
- SW_A_0: value 4,4 -> C2_R4
- SW_BACKSL_0: value C,5 -> CA_R4
- SW_BKSP_0: value D,7 -> CA_R5
- SW_B_0: value 7,2 -> C4_R2
- SW_CAPS_0: renamed from SW_LSHIFT_0; value 3,2 -> C1_R4
- SW_COLON_0: value A,4 -> C8_R3
- SW_COMMA_0: value 9,1 -> C7_R3
- SW_C_0: value 5,1 -> C3_R2
- SW_DEL_0: value D,5 -> CB_R5
- SW_DOWN_0: value D,1 -> CB_R1
- SW_D_0: value 5,3 -> C3_R4
- SW_END_0: value D,6 -> CB_R3
- SW_ENTER_0: value C,3 -> CA_R3
- SW_EQ_0: value B,6 -> C9_R6
- SW_ESC_0: value 1,6 -> C1_R8
- SW_E_0: value 5,4 -> C3_R5
- SW_F10_0: value A,7 -> C9_R7
- SW_F11_0: value B,7 -> CA_R8
- SW_F12_0: value C,7 -> CA_R7
- SW_F1_0: value 1,7 -> C2_R8
- SW_F2_0: value 2,7 -> C3_R8
- SW_F3_0: value 3,7 -> C4_R8
- SW_F4_0: value SW_F4_0 -> C5_R8
- SW_F5_0: value 5,7 -> C6_R8
- SW_F6_0: value 6,7 -> C7_R8
- SW_F7_0: value 7,7 -> C7_R7
- SW_F8_0: value 8,7 -> C8_R8
- SW_F9_0: value 9,7 -> C9_R8
- SW_F_0: value 6,3 -> C4_R4
- SW_G_0: value 7,4 -> C5_R4
- SW_HOME_0: value E,7 -> CB_R5
- SW_H_0: value 7,3 -> C5_R3
- SW_INS_0: value D,8 -> CB_R6
- SW_ISOBKSPX_0: value C,6 -> CA_R6
- SW_ISORSHIFT_0: value B,2 -> C9_R2
- SW_ISOXENTER_0: value B,4 -> C9_R3
- SW_I_0: value 9,3 -> C6_R5
- SW_JIS1_0: value 4,1 -> C3_R1
- SW_JIS2_0: value 8,1 -> C4_R1
- SW_JIS3_0: value 8,1 -> C6_R1
- SW_J_0: value 8,3 -> C6_R4
- SW_K_0: value 9,2 -> C6_R3
- SW_LBRAC_0: value B,5 -> C8_R4
- SW_LCTRL_0: renamed from SW_LALT_0; value 4,1 -> C1_R1
- SW_LEFT_0: value D,2 -> CA_R2
- SW_LSHIFTX_0: renamed from SW_LCTRL_0; value 3,1 -> C1_R2
- SW_LSHIFT_0: renamed from SW_ISOXLSHIFT_0; value 3,3 -> C1_R3
- SW_LSHIFT_1: renamed from SW_TAB_0; value 2,5 -> C1_R6
- SW_L_0: value A,3 -> C7_R4
- SW_MINUS_0: renamed from SW_DASH_0; value A,6 -> C8_R6
- SW_M_0: value 8,2 -> C6_R2
- SW_NUM0ISOX_0: value F,1 -> CD_R2
- SW_NUM0_0: value E,1 -> CD_R1
- SW_NUM1_0: value E,2 -> CC_R2
- SW_NUM2_0: value F,3 -> CD_R3
- SW_NUM3_0: value G,3 -> CE_R3
- SW_NUM4_0: value E,4 -> CC_R3
- SW_NUM5_0: value F,4 -> CD_R5
- SW_NUM6_0: value F,5 -> CD_R4
- SW_NUM7_0: value E,5 -> CC_R4
- SW_NUM8_0: value F,6 -> CD_R5
- SW_NUM9_0: value G,6 -> CD_R6
- SW_NUMASTR_0: value G,8 -> CE_R7
- SW_NUMDIV_0: value G,7 -> CE_R8
- SW_NUMENTISOX_0: value G,1 -> CE_R1
- SW_NUMEQ_0: value F,8 -> CD_R8
- SW_NUMLK_0: value F,7 -> CC_R6
- SW_NUMMIN_0: value G,5 -> CE_R6
- SW_NUMPER_0: value F,2 -> CE_R2
- SW_NUMPLS_0: renamed from SW_NUMPL_0; value G,4 -> CE_R5
- SW_N_0: value 7,1 -> C5_R2
- SW_O_0: value 9,4 -> C7_R5
- SW_PERIOD_0: value A,1 -> C7_R2
- SW_PGDN_0: value E,6 -> CC_R5
- SW_PGUP_0: value E,8 -> CC_R7
- SW_P_0: value A,5 -> C8_R5
- SW_Q_0: renamed from SW_W_0; value 4,5 -> C2_R6
- SW_RALT_1: value 8,1 -> C8_R1
- SW_RBRAC_0: value C,4 -> C9_R5
- SW_RCTRL_1: value C,1 -> CA_R1
- SW_RIGHT_0: value E,3 -> CC_R1
- SW_RSHIFT_0: value C,2 -> C9_R1
- SW_R_0: value 6,5 -> C4_R6
- SW_SLASH_0: value A,2 -> C8_R2
- SW_SPACE_0: value 6,1 -> C5_R1
- SW_S_0: value 4,3 -> C2_R3
- SW_TAB_1: renamed from SW_CAP_0; value 3,4 -> C1_R5
- SW_TICK_0: value 2,6 -> C1_R7
- SW_T_0: value 6,4 -> C4_R5
- SW_UP_0: value D,4 -> CB_R2
- SW_U_0: value 8,4 -> C6_R6
- SW_V_0: value 6,2 -> C4_R3
- SW_W_0: renamed from SW_Q_0; value 3,5 -> C2_R5
- SW_X_0: value 5,2 -> C3_R3
- SW_Y_0: value 7,5 -> C5_R5
- SW_Z_0: value 4,2 -> C2_R2
- moved SW_Z_0 73.2 mm to (141.0, 336.6)
- moved SW_DOWN_0 64.0 mm to (374.6, 324.9)
- moved SW_ESC_0 45.2 mm to (87.3, 156.7)
Connections:
- CAL1 pad COL: COL_B -> COL_A
- SWSW_NUMENT1 pad A: Net-(SWSW_NUMENT1-PadA) -> unconnected-(SWSW_NUMENT1-PadA)
- SWSW_NUMENT1 pad B: Net-(SWSW_NUMENT1-PadB) -> unconnected-(SWSW_NUMENT1-PadB)
- SWSW_NUMENT1 pad COL: COL_G -> COL_F
- SWSW_NUMENT1 pad REF: Net-(SWSW_NUMENT1-PadREF) -> unconnected-(SWSW_NUMENT1-PadREF)
- SW_0_0 pad A: Net-(SW_0_0-PadA) -> unconnected-(SW_0_0-PadA)
- SW_0_0 pad B: Net-(SW_0_0-PadB) -> unconnected-(SW_0_0-PadB)
- SW_0_0 pad COL: COL_9 -> COL_8
- SW_0_0 pad REF: Net-(SW_0_0-PadREF) -> unconnected-(SW_0_0-PadREF)
- SW_0_0 pad ROW: ROW_5 -> ROW_7
- SW_2_0 pad A: Net-(SW_1_0-PadA) -> unconnected-(SW_2_0-PadA)
- SW_2_0 pad B: Net-(SW_1_0-PadB) -> unconnected-(SW_2_0-PadB)
- SW_2_0 pad COL: COL_3 -> COL_2
- SW_2_0 pad REF: Net-(SW_1_0-PadREF) -> unconnected-(SW_2_0-PadREF)
- SW_2_0 pad ROW: ROW_6 -> ROW_7
- SW_3_0 pad A: Net-(SW_2_0-PadA) -> unconnected-(SW_3_0-PadA)
- SW_3_0 pad B: Net-(SW_2_0-PadB) -> unconnected-(SW_3_0-PadB)
- SW_3_0 pad COL: COL_4 -> COL_3
- SW_3_0 pad REF: Net-(SW_2_0-PadREF) -> unconnected-(SW_3_0-PadREF)
- SW_3_0 pad ROW: ROW_6 -> ROW_7
- SW_4_0 pad A: Net-(SW_4_0-PadA) -> unconnected-(SW_4_0-PadA)
- SW_4_0 pad B: Net-(SW_4_0-PadB) -> unconnected-(SW_4_0-PadB)
- SW_4_0 pad COL: COL_5 -> COL_3
- SW_4_0 pad REF: Net-(SW_4_0-PadREF) -> unconnected-(SW_4_0-PadREF)
- SW_4_0 pad ROW: ROW_5 -> ROW_6
- SW_5_0 pad A: Net-(SW_5_0-PadA) -> unconnected-(SW_5_0-PadA)
- SW_5_0 pad B: Net-(SW_5_0-PadB) -> unconnected-(SW_5_0-PadB)
- SW_5_0 pad COL: COL_6 -> COL_4
- SW_5_0 pad REF: Net-(SW_5_0-PadREF) -> unconnected-(SW_5_0-PadREF)
- SW_5_0 pad ROW: ROW_6 -> ROW_7
- SW_6_0 pad A: Net-(SW_6_0-PadA) -> unconnected-(SW_6_0-PadA)
- SW_6_0 pad B: Net-(SW_6_0-PadB) -> unconnected-(SW_6_0-PadB)
- SW_6_0 pad COL: COL_7 -> COL_5
- SW_6_0 pad REF: Net-(SW_6_0-PadREF) -> unconnected-(SW_6_0-PadREF)
- SW_6_0 pad ROW: ROW_6 -> ROW_7
- SW_7_0 pad A: Net-(SW_7_0-PadA) -> unconnected-(SW_7_0-PadA)
- SW_7_0 pad B: Net-(SW_7_0-PadB) -> unconnected-(SW_7_0-PadB)
- SW_7_0 pad COL: COL_8 -> COL_5
- SW_7_0 pad REF: Net-(SW_7_0-PadREF) -> unconnected-(SW_7_0-PadREF)
- SW_7_0 pad ROW: ROW_5 -> ROW_6
- SW_8_0 pad A: Net-(SW_8_0-PadA) -> unconnected-(SW_8_0-PadA)
- SW_8_0 pad B: Net-(SW_8_0-PadB) -> unconnected-(SW_8_0-PadB)
- SW_8_0 pad COL: COL_8 -> COL_6
- SW_8_0 pad REF: Net-(SW_8_0-PadREF) -> unconnected-(SW_8_0-PadREF)
- SW_8_0 pad ROW: ROW_6 -> ROW_7
- SW_9_0 pad A: Net-(SW_9_0-PadA) -> unconnected-(SW_9_0-PadA)
- SW_9_0 pad B: Net-(SW_9_0-PadB) -> unconnected-(SW_9_0-PadB)
- SW_9_0 pad COL: COL_9 -> COL_7
- SW_9_0 pad REF: Net-(SW_9_0-PadREF) -> unconnected-(SW_9_0-PadREF)
- SW_APOS_0 pad A: Net-(SW_APOS_0-PadA) -> unconnected-(SW_APOS_0-PadA)
- SW_APOS_0 pad B: Net-(SW_APOS_0-PadB) -> unconnected-(SW_APOS_0-PadB)
- SW_APOS_0 pad COL: COL_B -> COL_9
- SW_APOS_0 pad REF: Net-(SW_APOS_0-PadREF) -> unconnected-(SW_APOS_0-PadREF)
- SW_APOS_0 pad ROW: ROW_3 -> ROW_4
- SW_A_0 pad A: Net-(SW_A_0-PadA) -> unconnected-(SW_A_0-PadA)
- SW_A_0 pad B: Net-(SW_A_0-PadB) -> unconnected-(SW_A_0-PadB)
- SW_A_0 pad COL: COL_4 -> COL_2
- SW_A_0 pad REF: Net-(SW_A_0-PadREF) -> unconnected-(SW_A_0-PadREF)
- SW_BACKSL_0 pad A: Net-(SW_BACKSL_0-PadA) -> unconnected-(SW_BACKSL_0-PadA)
- SW_BACKSL_0 pad B: Net-(SW_BACKSL_0-PadB) -> unconnected-(SW_BACKSL_0-PadB)
- SW_BACKSL_0 pad COL: COL_C -> COL_A
- SW_BACKSL_0 pad REF: Net-(SW_BACKSL_0-PadREF) -> unconnected-(SW_BACKSL_0-PadREF)
- SW_BACKSL_0 pad ROW: ROW_5 -> ROW_4
- SW_BKSP_0 pad A: Net-(SW_BKSP_0-PadA) -> unconnected-(SW_BKSP_0-PadA)
- SW_BKSP_0 pad B: Net-(SW_BKSP_0-PadB) -> unconnected-(SW_BKSP_0-PadB)
- SW_BKSP_0 pad COL: COL_D -> COL_A
- SW_BKSP_0 pad REF: Net-(SW_BKSP_0-PadREF) -> unconnected-(SW_BKSP_0-PadREF)
- SW_BKSP_0 pad ROW: ROW_7 -> ROW_5
- SW_B_0 pad A: Net-(SW_B_0-PadA) -> unconnected-(SW_B_0-PadA)
- SW_B_0 pad B: Net-(SW_B_0-PadB) -> unconnected-(SW_B_0-PadB)
- SW_B_0 pad COL: COL_7 -> COL_4
- SW_B_0 pad REF: Net-(SW_B_0-PadREF) -> unconnected-(SW_B_0-PadREF)
- SW_CAPS_0 pad A: Net-(SW_LSHIFT_0-PadA) -> unconnected-(SW_CAPS_0-PadA)
- SW_CAPS_0 pad B: Net-(SW_LSHIFT_0-PadB) -> unconnected-(SW_CAPS_0-PadB)
- SW_CAPS_0 pad COL: COL_3 -> COL_1
- SW_CAPS_0 pad REF: Net-(SW_LSHIFT_0-PadREF) -> unconnected-(SW_CAPS_0-PadREF)
- SW_CAPS_0 pad ROW: ROW_2 -> ROW_4
- SW_COLON_0 pad A: Net-(SW_COLON_0-PadA) -> unconnected-(SW_COLON_0-PadA)
- SW_COLON_0 pad B: Net-(SW_COLON_0-PadB) -> unconnected-(SW_COLON_0-PadB)
- SW_COLON_0 pad COL: COL_A -> COL_8
- SW_COLON_0 pad REF: Net-(SW_COLON_0-PadREF) -> unconnected-(SW_COLON_0-PadREF)
- SW_COLON_0 pad ROW: ROW_4 -> ROW_3
- SW_COMMA_0 pad A: Net-(SW_COMMA_0-PadA) -> unconnected-(SW_COMMA_0-PadA)
- SW_COMMA_0 pad B: Net-(SW_COMMA_0-PadB) -> unconnected-(SW_COMMA_0-PadB)
- SW_COMMA_0 pad COL: COL_9 -> COL_7
- SW_COMMA_0 pad REF: Net-(SW_COMMA_0-PadREF) -> unconnected-(SW_COMMA_0-PadREF)
- SW_COMMA_0 pad ROW: ROW_1 -> ROW_3
- SW_C_0 pad A: Net-(SW_C_0-PadA) -> unconnected-(SW_C_0-PadA)
- SW_C_0 pad B: Net-(SW_C_0-PadB) -> unconnected-(SW_C_0-PadB)
- SW_C_0 pad COL: COL_5 -> COL_3
- SW_C_0 pad REF: Net-(SW_C_0-PadREF) -> unconnected-(SW_C_0-PadREF)
- SW_C_0 pad ROW: ROW_1 -> ROW_2
- SW_DEL_0 pad A: Net-(SW_DEL_0-PadA) -> unconnected-(SW_DEL_0-PadA)
- SW_DEL_0 pad B: Net-(SW_DEL_0-PadB) -> unconnected-(SW_DEL_0-PadB)
- SW_DEL_0 pad COL: COL_D -> COL_B
- SW_DEL_0 pad REF: Net-(SW_DEL_0-PadREF) -> unconnected-(SW_DEL_0-PadREF)
- SW_DOWN_0 pad A: Net-(SW_DOWN_0-PadA) -> unconnected-(SW_DOWN_0-PadA)
- SW_DOWN_0 pad B: Net-(SW_DOWN_0-PadB) -> unconnected-(SW_DOWN_0-PadB)
- SW_DOWN_0 pad COL: COL_D -> COL_B
- SW_DOWN_0 pad REF: Net-(SW_DOWN_0-PadREF) -> unconnected-(SW_DOWN_0-PadREF)
- SW_DOWN_0 pad ROW: ROW_1 -> ROW_2
- SW_D_0 pad A: Net-(SW_D_0-PadA) -> unconnected-(SW_D_0-PadA)
- SW_D_0 pad B: Net-(SW_D_0-PadB) -> unconnected-(SW_D_0-PadB)
- SW_D_0 pad COL: COL_5 -> COL_3
- SW_D_0 pad REF: Net-(SW_D_0-PadREF) -> unconnected-(SW_D_0-PadREF)
- SW_D_0 pad ROW: ROW_3 -> ROW_4
- SW_END_0 pad A: Net-(SW_END_0-PadA) -> unconnected-(SW_END_0-PadA)
- SW_END_0 pad B: Net-(SW_END_0-PadB) -> unconnected-(SW_END_0-PadB)
- SW_END_0 pad COL: COL_D -> COL_B
- SW_END_0 pad REF: Net-(SW_END_0-PadREF) -> unconnected-(SW_END_0-PadREF)
- SW_END_0 pad ROW: ROW_6 -> ROW_4
- SW_ENTER_0 pad A: Net-(SW_ENTER_0-PadA) -> unconnected-(SW_ENTER_0-PadA)
- SW_ENTER_0 pad B: Net-(SW_ENTER_0-PadB) -> unconnected-(SW_ENTER_0-PadB)
- SW_ENTER_0 pad COL: COL_C -> COL_A
- SW_ENTER_0 pad REF: Net-(SW_ENTER_0-PadREF) -> unconnected-(SW_ENTER_0-PadREF)
- SW_EQ_0 pad A: Net-(SW_EQ_0-PadA) -> unconnected-(SW_EQ_0-PadA)
- SW_EQ_0 pad B: Net-(SW_EQ_0-PadB) -> unconnected-(SW_EQ_0-PadB)
- SW_EQ_0 pad COL: COL_B -> COL_9
- SW_EQ_0 pad REF: Net-(SW_EQ_0-PadREF) -> unconnected-(SW_EQ_0-PadREF)
- SW_ESC_0 pad A: Net-(SW_ESC_0-PadA) -> unconnected-(SW_ESC_0-PadA)
- SW_ESC_0 pad B: Net-(SW_ESC_0-PadB) -> unconnected-(SW_ESC_0-PadB)
- SW_ESC_0 pad REF: Net-(SW_ESC_0-PadREF) -> unconnected-(SW_ESC_0-PadREF)
- SW_ESC_0 pad ROW: ROW_6 -> ROW_8
- SW_E_0 pad A: Net-(SW_E_0-PadA) -> unconnected-(SW_E_0-PadA)
- SW_E_0 pad B: Net-(SW_E_0-PadB) -> unconnected-(SW_E_0-PadB)
- SW_E_0 pad COL: COL_5 -> COL_3
- SW_E_0 pad REF: Net-(SW_E_0-PadREF) -> unconnected-(SW_E_0-PadREF)
- SW_E_0 pad ROW: ROW_4 -> ROW_5
- SW_F10_0 pad A: Net-(SW_F10_0-PadA) -> unconnected-(SW_F10_0-PadA)
- SW_F10_0 pad B: Net-(SW_F10_0-PadB) -> unconnected-(SW_F10_0-PadB)
- SW_F10_0 pad COL: COL_A -> COL_9
- SW_F10_0 pad REF: Net-(SW_F10_0-PadREF) -> unconnected-(SW_F10_0-PadREF)
- SW_F11_0 pad A: Net-(SW_F11_0-PadA) -> unconnected-(SW_F11_0-PadA)
- SW_F11_0 pad B: Net-(SW_F11_0-PadB) -> unconnected-(SW_F11_0-PadB)
- SW_F11_0 pad COL: COL_B -> COL_A
- SW_F11_0 pad REF: Net-(SW_F11_0-PadREF) -> unconnected-(SW_F11_0-PadREF)
- SW_F11_0 pad ROW: ROW_7 -> ROW_8
- SW_F12_0 pad A: Net-(SW_F12_0-PadA) -> unconnected-(SW_F12_0-PadA)
- SW_F12_0 pad B: Net-(SW_F12_0-PadB) -> unconnected-(SW_F12_0-PadB)
- SW_F12_0 pad COL: COL_C -> COL_A
- SW_F12_0 pad REF: Net-(SW_F12_0-PadREF) -> unconnected-(SW_F12_0-PadREF)
- SW_F1_0 pad A: Net-(SW_F1_0-PadA) -> unconnected-(SW_F1_0-PadA)
- SW_F1_0 pad B: Net-(SW_F1_0-PadB) -> unconnected-(SW_F1_0-PadB)
- SW_F1_0 pad COL: COL_1 -> COL_2
- SW_F1_0 pad REF: Net-(SW_F1_0-PadREF) -> unconnected-(SW_F1_0-PadREF)
- SW_F1_0 pad ROW: ROW_7 -> ROW_8
- SW_F2_0 pad A: Net-(SW_F2_0-PadA) -> unconnected-(SW_F2_0-PadA)
- SW_F2_0 pad B: Net-(SW_F2_0-PadB) -> unconnected-(SW_F2_0-PadB)
- SW_F2_0 pad COL: COL_2 -> COL_3
- SW_F2_0 pad REF: Net-(SW_F2_0-PadREF) -> unconnected-(SW_F2_0-PadREF)
- SW_F2_0 pad ROW: ROW_7 -> ROW_8
- SW_F3_0 pad A: Net-(SW_F3_0-PadA) -> unconnected-(SW_F3_0-PadA)
- SW_F3_0 pad B: Net-(SW_F3_0-PadB) -> unconnected-(SW_F3_0-PadB)
- SW_F3_0 pad COL: COL_3 -> COL_4
- SW_F3_0 pad REF: Net-(SW_F3_0-PadREF) -> unconnected-(SW_F3_0-PadREF)
- SW_F3_0 pad ROW: ROW_7 -> ROW_8
- SW_F4_0 pad A: Net-(SW_F4_0-PadA) -> unconnected-(SW_F4_0-PadA)
- SW_F4_0 pad B: Net-(SW_F4_0-PadB) -> unconnected-(SW_F4_0-PadB)
- SW_F4_0 pad COL: COL_4 -> COL_5
- SW_F4_0 pad REF: Net-(SW_F4_0-PadREF) -> unconnected-(SW_F4_0-PadREF)
- SW_F4_0 pad ROW: ROW_7 -> ROW_8
- SW_F5_0 pad A: Net-(SW_F5_0-PadA) -> unconnected-(SW_F5_0-PadA)
- SW_F5_0 pad B: Net-(SW_F5_0-PadB) -> unconnected-(SW_F5_0-PadB)
- SW_F5_0 pad COL: COL_5 -> COL_6
- SW_F5_0 pad REF: Net-(SW_F5_0-PadREF) -> unconnected-(SW_F5_0-PadREF)
- SW_F5_0 pad ROW: ROW_7 -> ROW_8
- SW_F6_0 pad A: Net-(SW_F6_0-PadA) -> unconnected-(SW_F6_0-PadA)
- SW_F6_0 pad B: Net-(SW_F6_0-PadB) -> unconnected-(SW_F6_0-PadB)
- SW_F6_0 pad COL: COL_6 -> COL_7
- SW_F6_0 pad REF: Net-(SW_F6_0-PadREF) -> unconnected-(SW_F6_0-PadREF)
- SW_F6_0 pad ROW: ROW_7 -> ROW_8
- SW_F7_0 pad A: Net-(SW_F7_0-PadA) -> unconnected-(SW_F7_0-PadA)
- SW_F7_0 pad B: Net-(SW_F7_0-PadB) -> unconnected-(SW_F7_0-PadB)
- SW_F7_0 pad REF: Net-(SW_F7_0-PadREF) -> unconnected-(SW_F7_0-PadREF)
- SW_F8_0 pad A: Net-(SW_F8_0-PadA) -> unconnected-(SW_F8_0-PadA)
- SW_F8_0 pad B: Net-(SW_F8_0-PadB) -> unconnected-(SW_F8_0-PadB)
- SW_F8_0 pad REF: Net-(SW_F8_0-PadREF) -> unconnected-(SW_F8_0-PadREF)
- SW_F8_0 pad ROW: ROW_7 -> ROW_8
- SW_F9_0 pad A: Net-(SW_F9_0-PadA) -> unconnected-(SW_F9_0-PadA)
- SW_F9_0 pad B: Net-(SW_F9_0-PadB) -> unconnected-(SW_F9_0-PadB)
- SW_F9_0 pad REF: Net-(SW_F9_0-PadREF) -> unconnected-(SW_F9_0-PadREF)
- SW_F9_0 pad ROW: ROW_7 -> ROW_8
- SW_F_0 pad A: Net-(SW_F_0-PadA) -> unconnected-(SW_F_0-PadA)
- SW_F_0 pad B: Net-(SW_F_0-PadB) -> unconnected-(SW_F_0-PadB)
- SW_F_0 pad COL: COL_6 -> COL_4
- SW_F_0 pad REF: Net-(SW_F_0-PadREF) -> unconnected-(SW_F_0-PadREF)
- SW_F_0 pad ROW: ROW_3 -> ROW_4
- SW_G_0 pad A: Net-(SW_G_0-PadA) -> unconnected-(SW_G_0-PadA)
- SW_G_0 pad B: Net-(SW_G_0-PadB) -> unconnected-(SW_G_0-PadB)
- SW_G_0 pad COL: COL_7 -> COL_5
- SW_G_0 pad REF: Net-(SW_G_0-PadREF) -> unconnected-(SW_G_0-PadREF)
- SW_HOME_0 pad A: Net-(SW_HOME_0-PadA) -> unconnected-(SW_HOME_0-PadA)
- SW_HOME_0 pad B: Net-(SW_HOME_0-PadB) -> unconnected-(SW_HOME_0-PadB)
- SW_HOME_0 pad COL: COL_E -> COL_B
- SW_HOME_0 pad REF: Net-(SW_HOME_0-PadREF) -> unconnected-(SW_HOME_0-PadREF)
- SW_HOME_0 pad ROW: ROW_7 -> ROW_6
- SW_H_0 pad A: Net-(SW_H_0-PadA) -> unconnected-(SW_H_0-PadA)
- SW_H_0 pad B: Net-(SW_H_0-PadB) -> unconnected-(SW_H_0-PadB)
- SW_H_0 pad COL: COL_7 -> COL_5
- SW_H_0 pad REF: Net-(SW_H_0-PadREF) -> unconnected-(SW_H_0-PadREF)
- SW_INS_0 pad A: Net-(SW_INS_0-PadA) -> unconnected-(SW_INS_0-PadA)
- SW_INS_0 pad B: Net-(SW_INS_0-PadB) -> unconnected-(SW_INS_0-PadB)
- SW_INS_0 pad COL: COL_D -> COL_B
- SW_INS_0 pad REF: Net-(SW_INS_0-PadREF) -> unconnected-(SW_INS_0-PadREF)
- SW_INS_0 pad ROW: ROW_8 -> ROW_7
- SW_ISOBKSPX_0 pad A: Net-(SW_ISOBKSPX_0-PadA) -> unconnected-(SW_ISOBKSPX_0-PadA)
- SW_ISOBKSPX_0 pad B: Net-(SW_ISOBKSPX_0-PadB) -> unconnected-(SW_ISOBKSPX_0-PadB)
- SW_ISOBKSPX_0 pad COL: COL_C -> COL_A
- SW_ISOBKSPX_0 pad REF: Net-(SW_ISOBKSPX_0-PadREF) -> unconnected-(SW_ISOBKSPX_0-PadREF)
- SW_ISORSHIFT_0 pad A: Net-(SW_ISORSHIFT_0-PadA) -> unconnected-(SW_ISORSHIFT_0-PadA)
- SW_ISORSHIFT_0 pad B: Net-(SW_ISORSHIFT_0-PadB) -> unconnected-(SW_ISORSHIFT_0-PadB)
- SW_ISORSHIFT_0 pad COL: COL_B -> COL_9
- SW_ISORSHIFT_0 pad REF: Net-(SW_ISORSHIFT_0-PadREF) -> unconnected-(SW_ISORSHIFT_0-PadREF)
- SW_ISOXENTER_0 pad A: Net-(SW_ISOXENTER_0-PadA) -> unconnected-(SW_ISOXENTER_0-PadA)
- SW_ISOXENTER_0 pad B: Net-(SW_ISOXENTER_0-PadB) -> unconnected-(SW_ISOXENTER_0-PadB)
- SW_ISOXENTER_0 pad COL: COL_B -> COL_9
- SW_ISOXENTER_0 pad REF: Net-(SW_ISOXENTER_0-PadREF) -> unconnected-(SW_ISOXENTER_0-PadREF)
- SW_ISOXENTER_0 pad ROW: ROW_4 -> ROW_3
- SW_I_0 pad A: Net-(SW_I_0-PadA) -> unconnected-(SW_I_0-PadA)
- SW_I_0 pad B: Net-(SW_I_0-PadB) -> unconnected-(SW_I_0-PadB)
- SW_I_0 pad COL: COL_9 -> COL_6
- SW_I_0 pad REF: Net-(SW_I_0-PadREF) -> unconnected-(SW_I_0-PadREF)
- SW_I_0 pad ROW: ROW_3 -> ROW_5
- SW_JIS1_0 pad A: Net-(SW_JIS1_0-PadA) -> unconnected-(SW_JIS1_0-PadA)
- SW_JIS1_0 pad B: Net-(SW_JIS1_0-PadB) -> unconnected-(SW_JIS1_0-PadB)
- SW_JIS1_0 pad COL: COL_4 -> COL_3
- SW_JIS1_0 pad REF: Net-(SW_JIS1_0-PadREF) -> unconnected-(SW_JIS1_0-PadREF)
- SW_JIS2_0 pad A: Net-(SW_JIS2_0-PadA) -> unconnected-(SW_JIS2_0-PadA)
- SW_JIS2_0 pad B: Net-(SW_JIS2_0-PadB) -> unconnected-(SW_JIS2_0-PadB)
- SW_JIS2_0 pad COL: COL_8 -> COL_4
- SW_JIS2_0 pad REF: Net-(SW_JIS2_0-PadREF) -> unconnected-(SW_JIS2_0-PadREF)
- SW_JIS3_0 pad A: Net-(SW_JIS3_0-PadA) -> unconnected-(SW_JIS3_0-PadA)
- SW_JIS3_0 pad B: Net-(SW_JIS3_0-PadB) -> unconnected-(SW_JIS3_0-PadB)
- SW_JIS3_0 pad COL: COL_8 -> COL_6
- SW_JIS3_0 pad REF: Net-(SW_JIS3_0-PadREF) -> unconnected-(SW_JIS3_0-PadREF)
- SW_J_0 pad A: Net-(SW_J_0-PadA) -> unconnected-(SW_J_0-PadA)
- SW_J_0 pad B: Net-(SW_J_0-PadB) -> unconnected-(SW_J_0-PadB)
- SW_J_0 pad COL: COL_8 -> COL_6
- SW_J_0 pad REF: Net-(SW_J_0-PadREF) -> unconnected-(SW_J_0-PadREF)
- SW_J_0 pad ROW: ROW_3 -> ROW_4
- SW_K_0 pad A: Net-(SW_K_0-PadA) -> unconnected-(SW_K_0-PadA)
- SW_K_0 pad B: Net-(SW_K_0-PadB) -> unconnected-(SW_K_0-PadB)
- SW_K_0 pad COL: COL_9 -> COL_6
- SW_K_0 pad REF: Net-(SW_K_0-PadREF) -> unconnected-(SW_K_0-PadREF)
- SW_K_0 pad ROW: ROW_2 -> ROW_3
- SW_LBRAC_0 pad A: Net-(SW_LBRAC_0-PadA) -> unconnected-(SW_LBRAC_0-PadA)
- SW_LBRAC_0 pad B: Net-(SW_LBRAC_0-PadB) -> unconnected-(SW_LBRAC_0-PadB)
- SW_LBRAC_0 pad COL: COL_B -> COL_8
- SW_LBRAC_0 pad REF: Net-(SW_LBRAC_0-PadREF) -> unconnected-(SW_LBRAC_0-PadREF)
- SW_LBRAC_0 pad ROW: ROW_5 -> ROW_4
- SW_LCTRL_0 pad A: Net-(SW_LALT_0-PadA) -> unconnected-(SW_LCTRL_0-PadA)
- SW_LCTRL_0 pad B: Net-(SW_LALT_0-PadB) -> unconnected-(SW_LCTRL_0-PadB)
- SW_LCTRL_0 pad COL: COL_4 -> COL_1
- SW_LCTRL_0 pad REF: Net-(SW_LALT_0-PadREF) -> unconnected-(SW_LCTRL_0-PadREF)
- SW_LEFT_0 pad A: Net-(SW_LEFT_0-PadA) -> unconnected-(SW_LEFT_0-PadA)
- SW_LEFT_0 pad B: Net-(SW_LEFT_0-PadB) -> unconnected-(SW_LEFT_0-PadB)
- SW_LEFT_0 pad COL: COL_D -> COL_B
- SW_LEFT_0 pad REF: Net-(SW_LEFT_0-PadREF) -> unconnected-(SW_LEFT_0-PadREF)
- SW_LEFT_0 pad ROW: ROW_2 -> ROW_1
- SW_LSHIFTX_0 pad A: Net-(SW_LCTRL_0-PadA) -> unconnected-(SW_LSHIFTX_0-PadA)
- SW_LSHIFTX_0 pad B: Net-(SW_LCTRL_0-PadB) -> unconnected-(SW_LSHIFTX_0-PadB)
- SW_LSHIFTX_0 pad COL: COL_3 -> COL_1
- SW_LSHIFTX_0 pad REF: Net-(SW_LCTRL_0-PadREF) -> unconnected-(SW_LSHIFTX_0-PadREF)
- SW_LSHIFTX_0 pad ROW: ROW_1 -> ROW_2
- SW_LSHIFT_0 pad A: Net-(SW_ISOXLSHIFT_0-PadA) -> unconnected-(SW_LSHIFT_0-PadA)
- SW_LSHIFT_0 pad B: Net-(SW_ISOXLSHIFT_0-PadB) -> unconnected-(SW_LSHIFT_0-PadB)
- SW_LSHIFT_0 pad COL: COL_3 -> COL_1
- SW_LSHIFT_0 pad REF: Net-(SW_ISOXLSHIFT_0-PadREF) -> unconnected-(SW_LSHIFT_0-PadREF)
- SW_LSHIFT_1 pad A: Net-(SW_TAB_0-PadA) -> unconnected-(SW_LSHIFT_1-PadA)
- SW_LSHIFT_1 pad B: Net-(SW_TAB_0-PadB) -> unconnected-(SW_LSHIFT_1-PadB)
- SW_LSHIFT_1 pad COL: Net-(SW_TAB_0-PadCOL) -> COL_1
- SW_LSHIFT_1 pad REF: Net-(SW_TAB_0-PadREF) -> unconnected-(SW_LSHIFT_1-PadREF)
- SW_LSHIFT_1 pad ROW: ROW_5 -> ROW_6
- SW_L_0 pad A: Net-(SW_L_0-PadA) -> unconnected-(SW_L_0-PadA)
- SW_L_0 pad B: Net-(SW_L_0-PadB) -> unconnected-(SW_L_0-PadB)
- SW_L_0 pad COL: COL_A -> COL_7
- SW_L_0 pad REF: Net-(SW_L_0-PadREF) -> unconnected-(SW_L_0-PadREF)
- SW_L_0 pad ROW: ROW_3 -> ROW_4
- SW_MINUS_0 pad A: Net-(SW_DASH_0-PadA) -> unconnected-(SW_MINUS_0-PadA)
- SW_MINUS_0 pad B: Net-(SW_DASH_0-PadB) -> unconnected-(SW_MINUS_0-PadB)
- SW_MINUS_0 pad COL: COL_A -> COL_8
- SW_MINUS_0 pad REF: Net-(SW_DASH_0-PadREF) -> unconnected-(SW_MINUS_0-PadREF)
- SW_M_0 pad A: Net-(SW_M_0-PadA) -> unconnected-(SW_M_0-PadA)
- SW_M_0 pad B: Net-(SW_M_0-PadB) -> unconnected-(SW_M_0-PadB)
- SW_M_0 pad COL: COL_8 -> COL_6
- SW_M_0 pad REF: Net-(SW_M_0-PadREF) -> unconnected-(SW_M_0-PadREF)
- SW_NUM0ISOX_0 pad A: Net-(SW_NUM0ISOX_0-PadA) -> unconnected-(SW_NUM0ISOX_0-PadA)
- SW_NUM0ISOX_0 pad B: Net-(SW_NUM0ISOX_0-PadB) -> unconnected-(SW_NUM0ISOX_0-PadB)
- SW_NUM0ISOX_0 pad COL: COL_F -> COL_D
- SW_NUM0ISOX_0 pad REF: Net-(SW_NUM0ISOX_0-PadREF) -> unconnected-(SW_NUM0ISOX_0-PadREF)
- SW_NUM0ISOX_0 pad ROW: ROW_1 -> ROW_2
- SW_NUM0_0 pad A: Net-(SW_NUM0_0-PadA) -> unconnected-(SW_NUM0_0-PadA)
- SW_NUM0_0 pad B: Net-(SW_NUM0_0-PadB) -> unconnected-(SW_NUM0_0-PadB)
- SW_NUM0_0 pad COL: COL_E -> COL_D
- SW_NUM0_0 pad REF: Net-(SW_NUM0_0-PadREF) -> unconnected-(SW_NUM0_0-PadREF)
- SW_NUM1_0 pad A: Net-(SW_NUM1_0-PadA) -> unconnected-(SW_NUM1_0-PadA)
- SW_NUM1_0 pad B: Net-(SW_NUM1_0-PadB) -> unconnected-(SW_NUM1_0-PadB)
- SW_NUM1_0 pad COL: COL_E -> COL_D
- SW_NUM1_0 pad REF: Net-(SW_NUM1_0-PadREF) -> unconnected-(SW_NUM1_0-PadREF)
- SW_NUM1_0 pad ROW: ROW_2 -> ROW_3
- SW_NUM2_0 pad A: Net-(SW_NUM2_0-PadA) -> unconnected-(SW_NUM2_0-PadA)
- SW_NUM2_0 pad B: Net-(SW_NUM2_0-PadB) -> unconnected-(SW_NUM2_0-PadB)
- SW_NUM2_0 pad COL: COL_F -> COL_E
- SW_NUM2_0 pad REF: Net-(SW_NUM2_0-PadREF) -> unconnected-(SW_NUM2_0-PadREF)
- SW_NUM2_0 pad ROW: ROW_3 -> ROW_2
- SW_NUM3_0 pad A: Net-(SW_NUM3_0-PadA) -> unconnected-(SW_NUM3_0-PadA)
- SW_NUM3_0 pad B: Net-(SW_NUM3_0-PadB) -> unconnected-(SW_NUM3_0-PadB)
- SW_NUM3_0 pad COL: COL_G -> COL_E
- SW_NUM3_0 pad REF: Net-(SW_NUM3_0-PadREF) -> unconnected-(SW_NUM3_0-PadREF)
- SW_NUM4_0 pad A: Net-(SW_NUM4_0-PadA) -> unconnected-(SW_NUM4_0-PadA)
- SW_NUM4_0 pad B: Net-(SW_NUM4_0-PadB) -> unconnected-(SW_NUM4_0-PadB)
- SW_NUM4_0 pad COL: COL_E -> COL_D
- SW_NUM4_0 pad REF: Net-(SW_NUM4_0-PadREF) -> unconnected-(SW_NUM4_0-PadREF)
- SW_NUM5_0 pad A: Net-(SW_NUM5_0-PadA) -> unconnected-(SW_NUM5_0-PadA)
- SW_NUM5_0 pad B: Net-(SW_NUM5_0-PadB) -> unconnected-(SW_NUM5_0-PadB)
- SW_NUM5_0 pad COL: COL_F -> COL_E
- SW_NUM5_0 pad REF: Net-(SW_NUM5_0-PadREF) -> unconnected-(SW_NUM5_0-PadREF)
- SW_NUM6_0 pad A: Net-(SW_NUM6_0-PadA) -> unconnected-(SW_NUM6_0-PadA)
- SW_NUM6_0 pad B: Net-(SW_NUM6_0-PadB) -> unconnected-(SW_NUM6_0-PadB)
- SW_NUM6_0 pad COL: COL_F -> COL_E
- SW_NUM6_0 pad REF: Net-(SW_NUM6_0-PadREF) -> unconnected-(SW_NUM6_0-PadREF)
- SW_NUM7_0 pad A: Net-(SW_NUM7_0-PadA) -> unconnected-(SW_NUM7_0-PadA)
- SW_NUM7_0 pad B: Net-(SW_NUM7_0-PadB) -> unconnected-(SW_NUM7_0-PadB)
- SW_NUM7_0 pad COL: COL_E -> COL_D
- SW_NUM7_0 pad REF: Net-(SW_NUM7_0-PadREF) -> unconnected-(SW_NUM7_0-PadREF)
- SW_NUM7_0 pad ROW: ROW_5 -> ROW_6
- SW_NUM8_0 pad A: Net-(SW_NUM8_0-PadA) -> unconnected-(SW_NUM8_0-PadA)
- SW_NUM8_0 pad B: Net-(SW_NUM8_0-PadB) -> unconnected-(SW_NUM8_0-PadB)
- SW_NUM8_0 pad COL: COL_F -> COL_D
- SW_NUM8_0 pad REF: Net-(SW_NUM8_0-PadREF) -> unconnected-(SW_NUM8_0-PadREF)
- SW_NUM8_0 pad ROW: ROW_6 -> ROW_5
- SW_NUM9_0 pad A: Net-(SW_NUM9_0-PadA) -> unconnected-(SW_NUM9_0-PadA)
- SW_NUM9_0 pad B: Net-(SW_NUM9_0-PadB) -> unconnected-(SW_NUM9_0-PadB)
- SW_NUM9_0 pad COL: COL_G -> COL_E
- SW_NUM9_0 pad REF: Net-(SW_NUM9_0-PadREF) -> unconnected-(SW_NUM9_0-PadREF)
- SW_NUM9_0 pad ROW: ROW_6 -> ROW_7
- SW_NUMASTR_0 pad A: Net-(SW_NUMASTR_0-PadA) -> unconnected-(SW_NUMASTR_0-PadA)
- SW_NUMASTR_0 pad B: Net-(SW_NUMASTR_0-PadB) -> unconnected-(SW_NUMASTR_0-PadB)
- SW_NUMASTR_0 pad COL: COL_G -> COL_F
- SW_NUMASTR_0 pad REF: Net-(SW_NUMASTR_0-PadREF) -> unconnected-(SW_NUMASTR_0-PadREF)
- SW_NUMDIV_0 pad A: Net-(SW_NUMDIV_0-PadA) -> unconnected-(SW_NUMDIV_0-PadA)
- SW_NUMDIV_0 pad B: Net-(SW_NUMDIV_0-PadB) -> unconnected-(SW_NUMDIV_0-PadB)
- SW_NUMDIV_0 pad COL: COL_G -> COL_E
- SW_NUMDIV_0 pad REF: Net-(SW_NUMDIV_0-PadREF) -> unconnected-(SW_NUMDIV_0-PadREF)
- SW_NUMDIV_0 pad ROW: ROW_7 -> ROW_8
- SW_NUMENTISOX_0 pad A: Net-(SW_NUMENTISOX_0-PadA) -> unconnected-(SW_NUMENTISOX_0-PadA)
- SW_NUMENTISOX_0 pad B: Net-(SW_NUMENTISOX_0-PadB) -> unconnected-(SW_NUMENTISOX_0-PadB)
- SW_NUMENTISOX_0 pad COL: COL_G -> COL_F
- SW_NUMENTISOX_0 pad REF: Net-(SW_NUMENTISOX_0-PadREF) -> unconnected-(SW_NUMENTISOX_0-PadREF)
- SW_NUMEQ_0 pad A: Net-(SW_NUMEQ_0-PadA) -> unconnected-(SW_NUMEQ_0-PadA)
- SW_NUMEQ_0 pad B: Net-(SW_NUMEQ_0-PadB) -> unconnected-(SW_NUMEQ_0-PadB)
- SW_NUMEQ_0 pad COL: COL_F -> COL_D
- SW_NUMEQ_0 pad REF: Net-(SW_NUMEQ_0-PadREF) -> unconnected-(SW_NUMEQ_0-PadREF)
- SW_NUMEQ_0 pad ROW: ROW_8 -> ROW_7
- SW_NUMLK_0 pad A: Net-(SW_NUMLK_0-PadA) -> unconnected-(SW_NUMLK_0-PadA)
- SW_NUMLK_0 pad B: Net-(SW_NUMLK_0-PadB) -> unconnected-(SW_NUMLK_0-PadB)
- SW_NUMLK_0 pad COL: COL_F -> COL_D
- SW_NUMLK_0 pad REF: Net-(SW_NUMLK_0-PadREF) -> unconnected-(SW_NUMLK_0-PadREF)
- SW_NUMLK_0 pad ROW: ROW_7 -> ROW_8
- SW_NUMMIN_0 pad A: Net-(SW_NUMMIN_0-PadA) -> unconnected-(SW_NUMMIN_0-PadA)
- SW_NUMMIN_0 pad B: Net-(SW_NUMMIN_0-PadB) -> unconnected-(SW_NUMMIN_0-PadB)
- SW_NUMMIN_0 pad COL: COL_G -> COL_E
- SW_NUMMIN_0 pad REF: Net-(SW_NUMMIN_0-PadREF) -> unconnected-(SW_NUMMIN_0-PadREF)
- SW_NUMMIN_0 pad ROW: ROW_5 -> ROW_6
- SW_NUMPER_0 pad A: Net-(SW_NUMPER_0-PadA) -> unconnected-(SW_NUMPER_0-PadA)
- SW_NUMPER_0 pad B: Net-(SW_NUMPER_0-PadB) -> unconnected-(SW_NUMPER_0-PadB)
- SW_NUMPER_0 pad COL: COL_F -> COL_E
- SW_NUMPER_0 pad REF: Net-(SW_NUMPER_0-PadREF) -> unconnected-(SW_NUMPER_0-PadREF)
- SW_NUMPER_0 pad ROW: ROW_2 -> ROW_1
- SW_NUMPLS_0 pad A: Net-(SW_NUMPL_0-PadA) -> unconnected-(SW_NUMPLS_0-PadA)
- SW_NUMPLS_0 pad B: Net-(SW_NUMPL_0-PadB) -> unconnected-(SW_NUMPLS_0-PadB)
- SW_NUMPLS_0 pad COL: COL_G -> COL_F
- SW_NUMPLS_0 pad REF: Net-(SW_NUMPL_0-PadREF) -> unconnected-(SW_NUMPLS_0-PadREF)
- SW_NUMPLS_0 pad ROW: ROW_4 -> ROW_5
- SW_N_0 pad A: Net-(SW_N_0-PadA) -> unconnected-(SW_N_0-PadA)
- SW_N_0 pad B: Net-(SW_N_0-PadB) -> unconnected-(SW_N_0-PadB)
- SW_N_0 pad COL: COL_7 -> COL_5
- SW_N_0 pad REF: Net-(SW_N_0-PadREF) -> unconnected-(SW_N_0-PadREF)
- SW_N_0 pad ROW: ROW_1 -> ROW_2
- SW_O_0 pad A: Net-(SW_O_0-PadA) -> unconnected-(SW_O_0-PadA)
- SW_O_0 pad B: Net-(SW_O_0-PadB) -> unconnected-(SW_O_0-PadB)
- SW_O_0 pad COL: COL_9 -> COL_7
- SW_O_0 pad REF: Net-(SW_O_0-PadREF) -> unconnected-(SW_O_0-PadREF)
- SW_O_0 pad ROW: ROW_4 -> ROW_5
- SW_PERIOD_0 pad A: Net-(SW_PERIOD_0-PadA) -> unconnected-(SW_PERIOD_0-PadA)
- SW_PERIOD_0 pad B: Net-(SW_PERIOD_0-PadB) -> unconnected-(SW_PERIOD_0-PadB)
- SW_PERIOD_0 pad COL: COL_A -> COL_7
- SW_PERIOD_0 pad REF: Net-(SW_PERIOD_0-PadREF) -> unconnected-(SW_PERIOD_0-PadREF)
- SW_PERIOD_0 pad ROW: ROW_1 -> ROW_2
- SW_PGDN_0 pad A: Net-(SW_PGDN_0-PadA) -> unconnected-(SW_PGDN_0-PadA)
- SW_PGDN_0 pad B: Net-(SW_PGDN_0-PadB) -> unconnected-(SW_PGDN_0-PadB)
- SW_PGDN_0 pad COL: COL_E -> COL_C
- SW_PGDN_0 pad REF: Net-(SW_PGDN_0-PadREF) -> unconnected-(SW_PGDN_0-PadREF)
- SW_PGDN_0 pad ROW: ROW_6 -> ROW_5
- SW_PGUP_0 pad A: Net-(SW_PGUP_0-PadA) -> unconnected-(SW_PGUP_0-PadA)
- SW_PGUP_0 pad B: Net-(SW_PGUP_0-PadB) -> unconnected-(SW_PGUP_0-PadB)
- SW_PGUP_0 pad COL: COL_E -> COL_C
- SW_PGUP_0 pad REF: Net-(SW_PGUP_0-PadREF) -> unconnected-(SW_PGUP_0-PadREF)
- SW_PGUP_0 pad ROW: ROW_8 -> ROW_6
- SW_P_0 pad A: Net-(SW_P_0-PadA) -> unconnected-(SW_P_0-PadA)
- SW_P_0 pad B: Net-(SW_P_0-PadB) -> unconnected-(SW_P_0-PadB)
- SW_P_0 pad COL: COL_A -> COL_8
- SW_P_0 pad REF: Net-(SW_P_0-PadREF) -> unconnected-(SW_P_0-PadREF)
- SW_Q_0 pad A: Net-(SW_W_0-PadA) -> unconnected-(SW_Q_0-PadA)
- SW_Q_0 pad B: Net-(SW_W_0-PadB) -> unconnected-(SW_Q_0-PadB)
- SW_Q_0 pad COL: COL_4 -> COL_2
- SW_Q_0 pad REF: Net-(SW_W_0-PadREF) -> unconnected-(SW_Q_0-PadREF)
- SW_Q_0 pad ROW: ROW_5 -> ROW_6
- SW_RALT_1 pad A: Net-(SW_RALT_1-PadA) -> unconnected-(SW_RALT_1-PadA)
- SW_RALT_1 pad B: Net-(SW_RALT_1-PadB) -> unconnected-(SW_RALT_1-PadB)
- SW_RALT_1 pad REF: Net-(SW_RALT_1-PadREF) -> unconnected-(SW_RALT_1-PadREF)
- SW_RBRAC_0 pad A: Net-(SW_RBRAC_0-PadA) -> unconnected-(SW_RBRAC_0-PadA)
- SW_RBRAC_0 pad B: Net-(SW_RBRAC_0-PadB) -> unconnected-(SW_RBRAC_0-PadB)
- SW_RBRAC_0 pad COL: COL_C -> COL_9
- SW_RBRAC_0 pad REF: Net-(SW_RBRAC_0-PadREF) -> unconnected-(SW_RBRAC_0-PadREF)
- SW_RBRAC_0 pad ROW: ROW_4 -> ROW_5
- SW_RCTRL_1 pad A: Net-(SW_RCTRL_1-PadA) -> unconnected-(SW_RCTRL_1-PadA)
- SW_RCTRL_1 pad B: Net-(SW_RCTRL_1-PadB) -> unconnected-(SW_RCTRL_1-PadB)
- SW_RCTRL_1 pad COL: COL_C -> COL_A
- SW_RCTRL_1 pad REF: Net-(SW_RCTRL_1-PadREF) -> unconnected-(SW_RCTRL_1-PadREF)
- SW_RCTRL_1 pad ROW: ROW_1 -> ROW_2
- SW_RIGHT_0 pad A: Net-(SW_RIGHT_0-PadA) -> unconnected-(SW_RIGHT_0-PadA)
- SW_RIGHT_0 pad B: Net-(SW_RIGHT_0-PadB) -> unconnected-(SW_RIGHT_0-PadB)
- SW_RIGHT_0 pad COL: COL_E -> COL_C
- SW_RIGHT_0 pad REF: Net-(SW_RIGHT_0-PadREF) -> unconnected-(SW_RIGHT_0-PadREF)
- SW_RIGHT_0 pad ROW: ROW_3 -> ROW_1
- SW_RSHIFT_0 pad A: Net-(SW_RSHIFT_0-PadA) -> unconnected-(SW_RSHIFT_0-PadA)
- SW_RSHIFT_0 pad B: Net-(SW_RSHIFT_0-PadB) -> unconnected-(SW_RSHIFT_0-PadB)
- SW_RSHIFT_0 pad COL: COL_C -> COL_9
- SW_RSHIFT_0 pad REF: Net-(SW_RSHIFT_0-PadREF) -> unconnected-(SW_RSHIFT_0-PadREF)
- SW_RSHIFT_0 pad ROW: ROW_2 -> ROW_1
- SW_R_0 pad A: Net-(SW_R_0-PadA) -> unconnected-(SW_R_0-PadA)
- SW_R_0 pad B: Net-(SW_R_0-PadB) -> unconnected-(SW_R_0-PadB)
- SW_R_0 pad COL: COL_6 -> COL_4
- SW_R_0 pad REF: Net-(SW_R_0-PadREF) -> unconnected-(SW_R_0-PadREF)
- SW_R_0 pad ROW: ROW_5 -> ROW_6
- SW_SLASH_0 pad A: Net-(SW_SLASH_0-PadA) -> unconnected-(SW_SLASH_0-PadA)
- SW_SLASH_0 pad B: Net-(SW_SLASH_0-PadB) -> unconnected-(SW_SLASH_0-PadB)
- SW_SLASH_0 pad COL: COL_A -> COL_8
- SW_SLASH_0 pad REF: Net-(SW_SLASH_0-PadREF) -> unconnected-(SW_SLASH_0-PadREF)
- SW_SPACE_0 pad A: Net-(SW_SPACE_0-PadA) -> unconnected-(SW_SPACE_0-PadA)
- SW_SPACE_0 pad B: Net-(SW_SPACE_0-PadB) -> unconnected-(SW_SPACE_0-PadB)
- SW_SPACE_0 pad COL: COL_6 -> COL_5
- SW_SPACE_0 pad REF: Net-(SW_SPACE_0-PadREF) -> unconnected-(SW_SPACE_0-PadREF)
- SW_S_0 pad A: Net-(SW_S_0-PadA) -> unconnected-(SW_S_0-PadA)
- SW_S_0 pad B: Net-(SW_S_0-PadB) -> unconnected-(SW_S_0-PadB)
- SW_S_0 pad COL: COL_4 -> COL_2
- SW_S_0 pad REF: Net-(SW_S_0-PadREF) -> unconnected-(SW_S_0-PadREF)
- SW_TAB_1 pad A: Net-(SW_CAP_0-PadA) -> unconnected-(SW_TAB_1-PadA)
- SW_TAB_1 pad B: Net-(SW_CAP_0-PadB) -> unconnected-(SW_TAB_1-PadB)
- SW_TAB_1 pad COL: COL_3 -> COL_1
- SW_TAB_1 pad REF: Net-(SW_CAP_0-PadREF) -> unconnected-(SW_TAB_1-PadREF)
- SW_TAB_1 pad ROW: ROW_4 -> ROW_5
- SW_TICK_0 pad A: Net-(SW_TICK_0-PadA) -> unconnected-(SW_TICK_0-PadA)
- SW_TICK_0 pad B: Net-(SW_TICK_0-PadB) -> unconnected-(SW_TICK_0-PadB)
- SW_TICK_0 pad COL: Net-(SW_TICK_0-PadCOL) -> COL_1
- SW_TICK_0 pad REF: Net-(SW_TICK_0-PadREF) -> unconnected-(SW_TICK_0-PadREF)
- SW_TICK_0 pad ROW: ROW_6 -> ROW_7
- SW_T_0 pad A: Net-(SW_T_0-PadA) -> unconnected-(SW_T_0-PadA)
- SW_T_0 pad B: Net-(SW_T_0-PadB) -> unconnected-(SW_T_0-PadB)
- SW_T_0 pad COL: COL_6 -> COL_4
- SW_T_0 pad REF: Net-(SW_T_0-PadREF) -> unconnected-(SW_T_0-PadREF)
- SW_T_0 pad ROW: ROW_4 -> ROW_5
- SW_UP_0 pad A: Net-(SW_UP_0-PadA) -> unconnected-(SW_UP_0-PadA)
- SW_UP_0 pad B: Net-(SW_UP_0-PadB) -> unconnected-(SW_UP_0-PadB)
- SW_UP_0 pad COL: COL_D -> COL_B
- SW_UP_0 pad REF: Net-(SW_UP_0-PadREF) -> unconnected-(SW_UP_0-PadREF)
- SW_UP_0 pad ROW: ROW_4 -> ROW_3
- SW_U_0 pad A: Net-(SW_U_0-PadA) -> unconnected-(SW_U_0-PadA)
- SW_U_0 pad B: Net-(SW_U_0-PadB) -> unconnected-(SW_U_0-PadB)
- SW_U_0 pad COL: COL_8 -> COL_6
- SW_U_0 pad REF: Net-(SW_U_0-PadREF) -> unconnected-(SW_U_0-PadREF)
- SW_U_0 pad ROW: ROW_4 -> ROW_6
- SW_V_0 pad A: Net-(SW_V_0-PadA) -> unconnected-(SW_V_0-PadA)
- SW_V_0 pad B: Net-(SW_V_0-PadB) -> unconnected-(SW_V_0-PadB)
- SW_V_0 pad COL: COL_6 -> COL_4
- SW_V_0 pad REF: Net-(SW_V_0-PadREF) -> unconnected-(SW_V_0-PadREF)
- SW_V_0 pad ROW: ROW_2 -> ROW_3
- SW_W_0 pad A: Net-(SW_Q_0-PadA) -> unconnected-(SW_W_0-PadA)
- SW_W_0 pad B: Net-(SW_Q_0-PadB) -> unconnected-(SW_W_0-PadB)
- SW_W_0 pad COL: COL_3 -> COL_2
- SW_W_0 pad REF: Net-(SW_Q_0-PadREF) -> unconnected-(SW_W_0-PadREF)
- SW_X_0 pad A: Net-(SW_X_0-PadA) -> unconnected-(SW_X_0-PadA)
- SW_X_0 pad B: Net-(SW_X_0-PadB) -> unconnected-(SW_X_0-PadB)
- SW_X_0 pad COL: COL_5 -> COL_3
- SW_X_0 pad REF: Net-(SW_X_0-PadREF) -> unconnected-(SW_X_0-PadREF)
- SW_X_0 pad ROW: ROW_2 -> ROW_3
- SW_Y_0 pad A: Net-(SW_Y_0-PadA) -> unconnected-(SW_Y_0-PadA)
- SW_Y_0 pad B: Net-(SW_Y_0-PadB) -> unconnected-(SW_Y_0-PadB)
- SW_Y_0 pad COL: COL_7 -> COL_5
- SW_Y_0 pad REF: Net-(SW_Y_0-PadREF) -> unconnected-(SW_Y_0-PadREF)
- SW_Z_0 pad A: Net-(SW_Z_0-PadA) -> unconnected-(SW_Z_0-PadA)
- SW_Z_0 pad B: Net-(SW_Z_0-PadB) -> unconnected-(SW_Z_0-PadB)
- SW_Z_0 pad COL: COL_4 -> COL_2
- SW_Z_0 pad REF: Net-(SW_Z_0-PadREF) -> unconnected-(SW_Z_0-PadREF)
Routing:
- net GND: track 9467.1 -> 976.4 mm
- net ROW_1: track 925.6 -> 222.3 mm
- net ROW_2: track 912.2 -> 224.6 mm
- net ROW_4: track 875.9 -> 190.1 mm
- net ROW_5: track 805.3 -> 128.6 mm
- net ROW_3: track 885.9 -> 209.5 mm
- net ROW_6: track 781.3 -> 122.6 mm
- net ROW_8: track 702.3 -> 62.5 mm
- net ROW_7: track 697.5 -> 59.6 mm
- net COL_8: track 333.1 -> 102.5 mm
- net COL_2: track 272.4 -> 52.8 mm
- net COL_1: track 289.8 -> 75.4 mm
- net COL_6: track 284.2 -> 71.8 mm
- net COL_4: track 248.0 -> 41.2 mm
- net COL_C: track 360.8 -> 163.7 mm
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Other:
- net class Default removed

Commit message: main details roughed out
Parts:
- removed SW_LSHIFT_1: C1_R6, lib_fp:SW_CAP_IBM_F_ALT
- added COL_1_TP9: C1_TestPoint, TestPoint:TestPoint_Pad_D1.0mm, B.Cu at (121.4, 295.7)
- added COL_2_TP10: C2_TestPoint, TestPoint:TestPoint_Pad_D1.0mm, B.Cu at (160.3, 295.7)
- added COL_3_TP11: C3_TestPoint, TestPoint:TestPoint_Pad_D1.0mm, B.Cu at (189.0, 295.4)
- added COL_4_TP12: C4_TestPoint, TestPoint:TestPoint_Pad_D1.0mm, B.Cu at (212.6, 295.1)
- added COL_5_TP13: C5_TestPoint, TestPoint:TestPoint_Pad_D1.0mm, B.Cu at (241.3, 295.1)
- added COL_6_TP14: C6_TestPoint, TestPoint:TestPoint_Pad_D1.0mm, B.Cu at (264.9, 295.4)
- added COL_7_TP15: C7_TestPoint, TestPoint:TestPoint_Pad_D1.0mm, B.Cu at (301.8, 295.1)
- added COL_8_TP16: C8_TestPoint, TestPoint:TestPoint_Pad_D1.0mm, B.Cu at (322.1, 295.7)
- added COL_9_TP17: C9_TestPoint, TestPoint:TestPoint_Pad_D1.0mm, B.Cu at (350.0, 295.1)
- added COL_A_TP18: CA_TestPoint, TestPoint:TestPoint_Pad_D1.0mm, B.Cu at (377.7, 295.9)
- added COL_B_TP19: CB_TestPoint, TestPoint:TestPoint_Pad_D1.0mm, B.Cu at (410.5, 295.4)
- added COL_C_TP20: CC_TestPoint, TestPoint:TestPoint_Pad_D1.0mm, B.Cu at (448.6, 294.9)
- added COL_D_TP21: CD_TestPoint, TestPoint:TestPoint_Pad_D1.0mm, B.Cu at (476.8, 294.9)
- added COL_E_TP22: CE_TestPoint, TestPoint:TestPoint_Pad_D1.0mm, B.Cu at (506.2, 294.9)
- added COL_F_TP23: CF_TestPoint, TestPoint:TestPoint_Pad_D1.0mm, B.Cu at (533.7, 295.7)
- added COL_G_TP24: CG_TestPoint, TestPoint:TestPoint_Pad_D1.0mm, B.Cu at (334.3, 137.4)
- added SW_1_0: C1_R6, lib_fp:SW_CAP_IBM_F_ALT, F.Cu at (131.3, 201.8)
- SWSW_NUMENT1, SW_0_0, SW_3_0, SW_6_0, SW_BACKSL_0, SW_COLON_0, SW_COMMA_0, SW_F11_0, SW_F1_0, SW_F5_0, SW_F9_0, SW_F_0, SW_INS_0, SW_LCTRL_0, SW_LSHIFT_0, SW_NUM0_0, SW_NUM1_0, SW_NUM4_0, SW_NUM7_0, SW_PGUP_0, SW_PRSC_0, SW_TICK_0, SW_V_0, SW_W_0: footprint lib_fp:SW_CAP_IBM_F_ALT -> lib_fp:SW_CAP_IBM_F
- SW_7_0, SW_9_0, SW_BKSP_0, SW_B_0, SW_F10_0, SW_F12_0, SW_HOME_0, SW_I_0, SW_LBRAC_0, SW_LSHIFTX_0, SW_L_0, SW_MINUS_0, SW_NUM0ISOX_0, SW_NUM3_0, SW_NUM8_0, SW_PERIOD_0, SW_RBRAC_0: footprint lib_fp:SW_CAP_IBM_F -> lib_fp:SW_CAP_IBM_F_ALT
- SW_JIS3_0: value C6_R1 -> C7_R1
- SW_JIS4_0: value C7_R1 -> C6_R1
- SW_NUM9_0: value CD_R6 -> CE_R7
- SW_NUMASTR_0: value CE_R7 -> CF_R8; footprint lib_fp:SW_CAP_IBM_F_ALT -> lib_fp:SW_CAP_IBM_F
- SW_NUMLK_0: value CC_R6 -> CC_R8
- SW_NUMMIN_0: value CE_R6 -> CF_R7; footprint lib_fp:SW_CAP_IBM_F_ALT -> lib_fp:SW_CAP_IBM_F
- moved H39 254.0 mm to (211.9, 352.7)
- moved H28 254.0 mm to (135.9, 352.7)
- moved H32 254.0 mm to (173.9, 352.7)
- moved H9 247.9 mm to (193.4, 365.2)
- moved H19 240.5 mm to (148.8, 367.0)
- moved SW_SCLK_0 218.4 mm to (425.3, 159.8)
- moved SW_PRSC_0 217.6 mm to (406.3, 159.8)
- moved SW_PAUS_0 210.3 mm to (444.3, 159.8)
- moved H3 188.5 mm to (158.8, 360.1)
- moved SW_LALT_0 188.3 mm to (164.6, 285.8)
- moved H1 172.7 mm to (172.0, 361.0)
- moved H4 172.7 mm to (191.0, 340.0)
- moved H2 151.6 mm to (164.4, 381.1)
- moved H5 151.6 mm to (183.4, 360.1)
- moved H6 142.5 mm to (158.6, 410.7)
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Connections:
- CAL1 pad COL: COL_A -> COL_9
- SWSW_NUMENT1 pad ROW: ROW_2 -> ROW_3
- SW_NUMMIN_0 pad COL: COL_E -> unconnected-(SW_NUMMIN_0-PadCOL)
- SW_NUMMIN_0 pad ROW: ROW_6 -> ROW_7
- SW_RCTRL_1 pad ROW: ROW_2 -> ROW_1
- SW_RSHIFT_0 pad COL: COL_9 -> COL_A
- SW_RSHIFT_0 pad ROW: ROW_1 -> ROW_2
Routing:
- net GND: track 976.4 -> 8.65 mm, vias 0 -> 4
- net ROW_7: track 59.6 -> 963.6 mm
- net ROW_1: track 222.3 -> 948.6 mm
- net ROW_5: track 128.6 -> 819.1 mm
- net ROW_4: track 190.1 -> 852.2 mm
- net ROW_3: track 209.5 -> 856.6 mm
- net ROW_6: track 122.6 -> 749.4 mm
- net ROW_8: track 62.5 -> 664.0 mm
- net ROW_2: track 224.6 -> 796.5 mm
- net COL_G: track 358.1 -> 5.07 mm
- net COL_4: track 41.2 -> 297.7 mm
- net COL_1: track 75.4 -> 330.1 mm
- net COL_2: track 52.8 -> 300.3 mm
- net COL_3: track 46.5 -> 293.8 mm
- net COL_5: track 48.2 -> 261.9 mm
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Other:
- board size 500 x 194 mm -> 463.1 x 170.8 mm
- board text added: "CC"
- board text removed: "IBM-M122-CAP Rev. 2 #:"
- board text removed: "made w/ <3 by ViviLazuli, 2020"

Commit message: updates
Routing:
- net GND: track 8.65 -> 178.9 mm, vias 4 -> 76

Commit message: save progress
Parts:
- moved H44 350.3 mm to (48.5, 49.6)
- moved H45 350.3 mm to (71.9, 70.6)
- moved H46 350.3 mm to (76.5, 91.6)
- moved H50 350.3 mm to (95.4, 49.6)
- moved H51 350.3 mm to (114.4, 91.6)
- moved H54 350.3 mm to (133.5, 49.6)
- moved H56 350.3 mm to (142.5, 70.6)
- moved H57 350.3 mm to (161.5, 91.6)
- moved H59 350.3 mm to (180.5, 49.6)
- moved H60 350.3 mm to (218.5, 91.6)
- moved H47 331.7 mm to (128.9, 58.8)
- moved H48 331.7 mm to (128.9, 79.8)
- moved H49 331.7 mm to (128.9, 99.8)
- moved H52 331.7 mm to (166.9, 58.8)
- moved H53 331.7 mm to (166.9, 79.8)
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Connections:
- SW_NUMMIN_0 pad COL: unconnected-(SW_NUMMIN_0-PadCOL) -> COL_F
Routing:
- net ROW_1: track 948.6 -> 794.4 mm
- net COL_E: track 404.4 -> 362.4 mm
- net ROW_4: track 852.2 -> 818.9 mm
- net ROW_2: track 796.5 -> 767.8 mm
- net ROW_5: track 819.1 -> 791.0 mm
- net ROW_3: track 856.7 -> 835.8 mm
- net COL_4: track 297.7 -> 277.6 mm
- net COL_7: track 218.2 -> 204.8 mm
- net ROW_7: track 963.6 -> 975.0 mm
- net COL_5: track 261.9 -> 251.3 mm
- net ROW_8: track 664.0 -> 674.1 mm
- net COL_A: track 232.9 -> 224.0 mm
- net GND: track 178.9 -> 170.3 mm, vias 76 -> 72
- net COL_9: track 201.6 -> 194.5 mm
- net COL_3: track 293.8 -> 287.2 mm
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Other:
- board size 463.1 x 170.8 mm -> 463.2 x 170.8 mm
