File: mtfjis.kicad_pcb (KiCad board)
At the start: 2 copper layers, 463.2 x 170.8 mm, 201 parts, among them J1 CONN_CAP_IBM_F

Commit message: updates
Routing:
- net ROW_8: track 674.1 -> 693.4 mm
- net COL_9: track 194.5 -> 204.4 mm
- net COL_B: track 275.2 -> 283.2 mm
- net COL_3: track 287.2 -> 279.3 mm
- net COL_7: track 204.8 -> 199.4 mm
- net COL_D: track 334.0 -> 339.3 mm
- net COL_A: track 224.0 -> 229.1 mm
- net COL_6: track 237.8 -> 234.2 mm
- net COL_2: track 296.2 -> 292.7 mm
- net COL_1: track 332.5 -> 329.6 mm
- net COL_E: track 362.4 -> 364.7 mm
- net COL_F: track 350.8 -> 352.7 mm
- net COL_5: track 251.3 -> 253.1 mm
- net ROW_1: track 794.4 -> 792.6 mm
- net ROW_3: track 835.8 -> 834.0 mm
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Other:
- outline, holes or cut-outs redrawn

Commit message: update
Parts:
- moved ROW_8_TP8 6.73 mm to (463.0, -102.1)
Routing:
- net ROW_8: track 693.4 -> 689.9 mm
Other:
- board text added: "ibm model m-to-f jis pcb thingy"
- board text added: "thanks to idollar vivi purdeaandrei and andj00"
