File: mtfjis.kicad_sch (KiCad schematic)
At the start: 199 parts, among them J1 CONN_CAP_IBM_F

Commit message: gitignore mtfjis-backups, wipe tracks and update schematic
Parts:
- removed SW_3_0: 5,6, lib_fp:SW_CAP_IBM_F, symbol lib_sch:SW_CAP_IBM_F
- removed SW_DOWN_0: D,1, lib_fp:SW_CAP_IBM_F_ALT, symbol lib_sch:SW_CAP_IBM_F
- added SW_LALT_0: C2_R1, lib_fp:SW_CAP_IBM_F_ALT, symbol lib_sch:SW_CAP_IBM_F
- added SW_PAUS_0: CC_R8, lib_fp:SW_CAP_IBM_F_ALT, symbol lib_sch:SW_CAP_IBM_F
- added SW_PRSC_0: CB_R8, lib_fp:SW_CAP_IBM_F_ALT, symbol lib_sch:SW_CAP_IBM_F
- added SW_SCLK_0: CB_R7, lib_fp:SW_CAP_IBM_F, symbol lib_sch:SW_CAP_IBM_F
- SWSW_NUMENT1: value G,2 -> CE_R4
- SW_0_0: value 9,5 -> C8_R7
- SW_2_0: renamed from SW_1_0; value 3,6 -> C2_R7
- SW_3_0: renamed from SW_2_0; value 4,6 -> C3_R7
- SW_4_0: value 5,5 -> C3_R6
- SW_5_0: value 6,6 -> C4_R7
- SW_6_0: value 7,6 -> C5_R7
- SW_7_0: value 8,5 -> C5_R6
- SW_8_0: value 8,6 -> C6_R7
- SW_9_0: value 9,6 -> C7_R6
- SW_APOS_0: value B,3 -> C9_R4
- SW_A_0: value 4,4 -> C2_R4
- SW_BACKSL_0: value C,5 -> CA_R4
- SW_BKSP_0: value D,7 -> CA_R5
- SW_B_0: value 7,2 -> C4_R2
- SW_COLON_0: value A,4 -> C8_R3
- SW_COMMA_0: value 9,1 -> C7_R3
- SW_C_0: value 5,1 -> C3_R2
- SW_DEL_0: value D,5 -> CB_R5
- SW_DOWN_0: renamed from SW_CENTER_0; value D,3 -> CB_R1
- SW_D_0: value 5,3 -> C3_R4
- SW_END_0: value D,6 -> CB_R3
- SW_ENTER_0: value C,3 -> CA_R3
- SW_EQ_0: value B,6 -> C9_R6
- SW_E_0: value 5,4 -> C3_R5
- SW_F10_0: value A,7 -> C9_R7
- SW_F11_0: value B,7 -> CA_R8
- SW_F12_0: value C,7 -> CA_R7
- SW_F1_0: value 1,7 -> C2_R8
- SW_F2_0: value 2,7 -> C3_R8
- SW_F3_0: value 3,7 -> C4_R8
- SW_F4_0: value SW_F4_0 -> C5_R8
- SW_F5_0: value 5,7 -> C6_R8
- SW_F6_0: value 6,7 -> C7_R8
- SW_F7_0: value 7,7 -> C7_R7
- SW_F8_0: value 8,7 -> C8_R8
- SW_F9_0: value 9,7 -> C9_R8
- SW_F_0: value 6,3 -> C4_R4
- SW_G_0: value 7,4 -> C5_R4
- SW_HOME_0: value E,7 -> CB_R5
- SW_H_0: value 7,3 -> C5_R3
- SW_INS_0: value D,8 -> CB_R6
- SW_ISOBKSPX_0: value C,6 -> CA_R6
- SW_ISORSHIFT_0: value B,2 -> C9_R2
- SW_ISOXENTER_0: value B,4 -> C9_R3
- SW_I_0: value 9,3 -> C6_R5
- SW_JIS1_0: value 4,1 -> C3_R1
- SW_JIS2_0: value 4,1 -> C4_R1
- SW_JIS3_0: value 8,1 -> C6_R1
- SW_JIS4_0: value 8,1 -> C7_R1
- SW_J_0: value 8,3 -> C6_R4
- SW_K_0: value 9,2 -> C6_R3
- SW_LBRAC_0: value B,5 -> C8_R4
- SW_LEFT_0: value D,2 -> CA_R2
- SW_L_0: value A,3 -> C7_R4
- SW_MINUS_0: renamed from SW_DASH_0; value A,6 -> C8_R6
- SW_M_0: value 8,2 -> C6_R2
- SW_NUM0ISOX_0: value F,1 -> CD_R2
- SW_NUM0_0: value E,1 -> CD_R1
- SW_NUM1_0: value E,2 -> CC_R2
- SW_NUM2_0: value F,3 -> CD_R3
- SW_NUM3_0: value G,3 -> CE_R3
- SW_NUM4_0: value E,4 -> CC_R3
- SW_NUM5_0: value F,4 -> CD_R5
- SW_NUM6_0: value F,5 -> CD_R4
- SW_NUM7_0: value E,5 -> CC_R4
- SW_NUM8_0: value F,6 -> CD_R5
- SW_NUM9_0: value G,6 -> CD_R6
- SW_NUMASTR_0: value G,8 -> CE_R7
- SW_NUMDIV_0: value G,7 -> CE_R8
- SW_NUMENTISOX_0: value G,1 -> CE_R1
- SW_NUMEQ_0: value F,8 -> CD_R8
- SW_NUMLK_0: value F,7 -> CC_R6
- SW_NUMMIN_0: value G,5 -> CE_R6
- SW_NUMPER_0: value F,2 -> CE_R2
- SW_NUMPLS_0: renamed from SW_NUMPL_0; value G,4 -> CE_R5
- SW_N_0: value 7,1 -> C5_R2
- SW_O_0: value 9,4 -> C7_R5
- SW_PERIOD_0: value A,1 -> C7_R2
- SW_PGDN_0: value E,6 -> CC_R5
- SW_PGUP_0: value E,8 -> CC_R7
- SW_P_0: value A,5 -> C8_R5
- SW_Q_0: renamed from SW_W_0; value 4,5 -> C2_R6
- SW_RALT_1: value 8,1 -> C8_R1
- SW_RBRAC_0: value C,4 -> C9_R5
- SW_RCTRL_1: value C,1 -> CA_R1
- SW_RIGHT_0: value E,3 -> CC_R1
- SW_RSHIFT_0: value C,2 -> C9_R1
- SW_R_0: value 6,5 -> C4_R6
- SW_SLASH_0: value A,2 -> C8_R2
- SW_SPACE_0: value 6,1 -> C5_R1
- SW_S_0: value 4,3 -> C2_R3
- SW_TAB_1: renamed from SW_CAP_0; value C1_R6 -> C1_R5
- SW_T_0: value 6,4 -> C4_R5
- SW_UP_0: value D,4 -> CB_R2
- SW_U_0: value 8,4 -> C6_R6
- SW_V_0: value 6,2 -> C4_R3
- SW_W_0: renamed from SW_Q_0; value 3,5 -> C2_R5
- SW_X_0: value 5,2 -> C3_R3
- SW_Y_0: value 7,5 -> C5_R5
- SW_Z_0: value 4,2 -> C2_R2
- renumbered SW_LSHIFT_0 to SW_CAPS_0, SW_LALT_0 to SW_LCTRL_0, SW_LCTRL_0 to SW_LSHIFTX_0, SW_ISOXLSHIFT_0 to SW_LSHIFT_0, SW_TAB_0 to SW_LSHIFT_1
Connections:
- net COL_1: now also SW_LSHIFT_1.COL, SW_TICK_0.COL
- net COL_2: now also SW_LALT_0.COL; no longer SW_X_0.COL
- net COL_3: now also SW_4_0.COL, SW_X_0.COL; no longer SW_F3_0.COL, SW_JIS2_0.COL
- net COL_4: now also SW_5_0.COL, SW_B_0.COL, SW_F3_0.COL, SW_F_0.COL, SW_JIS2_0.COL, SW_R_0.COL, SW_T_0.COL, SW_V_0.COL; no longer SW_F4_0.COL
- net COL_5: now also SW_6_0.COL, SW_7_0.COL, SW_F4_0.COL, SW_G_0.COL, SW_H_0.COL, SW_N_0.COL, SW_SPACE_0.COL, SW_Y_0.COL; no longer SW_4_0.COL, SW_F5_0.COL
- net COL_6: now also SW_8_0.COL, SW_F5_0.COL, SW_I_0.COL, SW_JIS3_0.COL, SW_J_0.COL, SW_K_0.COL, SW_M_0.COL, SW_U_0.COL; no longer SW_5_0.COL, SW_F6_0.COL, SW_F_0.COL, SW_R_0.COL, SW_SPACE_0.COL, SW_T_0.COL, SW_V_0.COL
- net COL_7: now also SW_9_0.COL, SW_COMMA_0.COL, SW_F6_0.COL, SW_JIS4_0.COL, SW_L_0.COL, SW_O_0.COL, SW_PERIOD_0.COL; no longer SW_6_0.COL, SW_B_0.COL, SW_G_0.COL, SW_H_0.COL, SW_N_0.COL, SW_Y_0.COL
- net COL_8: now also SW_0_0.COL, SW_COLON_0.COL, SW_LBRAC_0.COL, SW_MINUS_0.COL, SW_P_0.COL, SW_SLASH_0.COL; no longer SW_7_0.COL, SW_8_0.COL, SW_JIS3_0.COL, SW_JIS4_0.COL, SW_J_0.COL, SW_M_0.COL, SW_U_0.COL
- net COL_9: now also SW_APOS_0.COL, SW_EQ_0.COL, SW_F10_0.COL, SW_ISORSHIFT_0.COL, SW_ISOXENTER_0.COL, SW_RBRAC_0.COL, SW_RSHIFT_0.COL; no longer SW_0_0.COL, SW_9_0.COL, SW_COMMA_0.COL, SW_I_0.COL, SW_K_0.COL, SW_O_0.COL
- net COL_A: now also CAL1.COL, SW_BACKSL_0.COL, SW_BKSP_0.COL, SW_ENTER_0.COL, SW_F11_0.COL, SW_F12_0.COL, SW_ISOBKSPX_0.COL, SW_RCTRL_1.COL; no longer SW_COLON_0.COL, SW_F10_0.COL, SW_L_0.COL, SW_MINUS_0.COL, SW_PERIOD_0.COL, SW_P_0.COL, SW_SLASH_0.COL
- net COL_B: now also SW_DEL_0.COL, SW_DOWN_0.COL, SW_END_0.COL, SW_HOME_0.COL, SW_INS_0.COL, SW_LEFT_0.COL, SW_UP_0.COL, SW_PRSC_0.COL; no longer CAL1.COL, SW_APOS_0.COL, SW_EQ_0.COL, SW_F11_0.COL, SW_ISORSHIFT_0.COL, SW_ISOXENTER_0.COL, SW_LBRAC_0.COL
- net COL_C: now also SW_PGDN_0.COL, SW_PGUP_0.COL, SW_RIGHT_0.COL, SW_PAUS_0.COL, SW_SCLK_0.COL; no longer SW_BACKSL_0.COL, SW_ENTER_0.COL, SW_F12_0.COL, SW_ISOBKSPX_0.COL, SW_RBRAC_0.COL, SW_RCTRL_1.COL, SW_RSHIFT_0.COL
- net COL_D: now also SW_NUM0ISOX_0.COL, SW_NUM0_0.COL, SW_NUM1_0.COL, SW_NUM4_0.COL, SW_NUM7_0.COL, SW_NUM8_0.COL, SW_NUMEQ_0.COL, SW_NUMLK_0.COL; no longer SW_BKSP_0.COL, SW_DEL_0.COL, SW_DOWN_0.COL, SW_END_0.COL, SW_INS_0.COL, SW_LEFT_0.COL, SW_UP_0.COL
- net COL_E: now also SW_NUM2_0.COL, SW_NUM3_0.COL, SW_NUM5_0.COL, SW_NUM6_0.COL, SW_NUM9_0.COL, SW_NUMDIV_0.COL, SW_NUMMIN_0.COL, SW_NUMPER_0.COL; no longer SW_HOME_0.COL, SW_NUM0_0.COL, SW_NUM1_0.COL, SW_NUM4_0.COL, SW_NUM7_0.COL, SW_PGDN_0.COL, SW_PGUP_0.COL, SW_RIGHT_0.COL
- net COL_F: now also SWSW_NUMENT1.COL, SW_NUMASTR_0.COL, SW_NUMENTISOX_0.COL, SW_NUMPLS_0.COL; no longer SW_NUM0ISOX_0.COL, SW_NUM2_0.COL, SW_NUM5_0.COL, SW_NUM6_0.COL, SW_NUM8_0.COL, SW_NUMEQ_0.COL, SW_NUMLK_0.COL, SW_NUMPER_0.COL
- net COL_G: no longer SWSW_NUMENT1.COL, SW_NUM3_0.COL, SW_NUM9_0.COL, SW_NUMASTR_0.COL, SW_NUMDIV_0.COL, SW_NUMENTISOX_0.COL, SW_NUMMIN_0.COL, SW_NUMPLS_0.COL
- net ROW_1: now also SW_LEFT_0.ROW, SW_NUMPER_0.ROW, SW_RIGHT_0.ROW, SW_RSHIFT_0.ROW, SW_LALT_0.ROW; no longer SW_COMMA_0.ROW, SW_NUM0ISOX_0.ROW, SW_N_0.ROW, SW_PERIOD_0.ROW, SW_RCTRL_1.ROW, SW_X_0.ROW
- net ROW_2: now also SW_DOWN_0.ROW, SW_NUM0ISOX_0.ROW, SW_NUM2_0.ROW, SW_N_0.ROW, SW_PERIOD_0.ROW, SW_RCTRL_1.ROW; no longer SW_K_0.ROW, SW_LEFT_0.ROW, SW_NUM1_0.ROW, SW_NUMPER_0.ROW, SW_RSHIFT_0.ROW, SW_V_0.ROW
- net ROW_3: now also SW_COLON_0.ROW, SW_COMMA_0.ROW, SW_ISOXENTER_0.ROW, SW_K_0.ROW, SW_NUM1_0.ROW, SW_UP_0.ROW, SW_V_0.ROW, SW_X_0.ROW; no longer SW_APOS_0.ROW, SW_DOWN_0.ROW, SW_D_0.ROW, SW_F_0.ROW, SW_I_0.ROW, SW_J_0.ROW, SW_L_0.ROW, SW_NUM2_0.ROW, SW_RIGHT_0.ROW
- net ROW_4: now also SW_APOS_0.ROW, SW_BACKSL_0.ROW, SW_D_0.ROW, SW_END_0.ROW, SW_F_0.ROW, SW_J_0.ROW, SW_LBRAC_0.ROW, SW_L_0.ROW; no longer SW_COLON_0.ROW, SW_E_0.ROW, SW_ISOXENTER_0.ROW, SW_NUMPLS_0.ROW, SW_O_0.ROW, SW_RBRAC_0.ROW, SW_T_0.ROW, SW_UP_0.ROW, SW_U_0.ROW
- net ROW_5: now also SW_BKSP_0.ROW, SW_E_0.ROW, SW_I_0.ROW, SW_NUM8_0.ROW, SW_NUMPLS_0.ROW, SW_O_0.ROW, SW_PGDN_0.ROW, SW_RBRAC_0.ROW, SW_T_0.ROW; no longer SW_0_0.ROW, SW_3_0.ROW, SW_4_0.ROW, SW_7_0.ROW, SW_BACKSL_0.ROW, SW_LBRAC_0.ROW, SW_NUM7_0.ROW, SW_NUMMIN_0.ROW, SW_R_0.ROW
- net ROW_6: now also SW_4_0.ROW, SW_7_0.ROW, SW_HOME_0.ROW, SW_NUM7_0.ROW, SW_NUMMIN_0.ROW, SW_PGUP_0.ROW, SW_R_0.ROW, SW_U_0.ROW; no longer SW_5_0.ROW, SW_6_0.ROW, SW_8_0.ROW, SW_END_0.ROW, SW_NUM8_0.ROW, SW_NUM9_0.ROW, SW_PGDN_0.ROW
- net ROW_7: now also SW_0_0.ROW, SW_3_0.ROW, SW_5_0.ROW, SW_6_0.ROW, SW_8_0.ROW, SW_INS_0.ROW, SW_NUM9_0.ROW, SW_NUMEQ_0.ROW, SW_PAUS_0.ROW; no longer SW_BKSP_0.ROW, SW_F11_0.ROW, SW_F3_0.ROW, SW_F4_0.ROW, SW_F5_0.ROW, SW_F6_0.ROW, SW_F8_0.ROW, SW_F9_0.ROW, SW_HOME_0.ROW, SW_NUMDIV_0.ROW, SW_NUMLK_0.ROW
- net ROW_8: now also SW_F11_0.ROW, SW_F3_0.ROW, SW_F4_0.ROW, SW_F5_0.ROW, SW_F6_0.ROW, SW_F8_0.ROW, SW_F9_0.ROW, SW_NUMDIV_0.ROW, SW_NUMLK_0.ROW, SW_PRSC_0.ROW, SW_SCLK_0.ROW; no longer SW_INS_0.ROW, SW_NUMEQ_0.ROW, SW_PGUP_0.ROW
Other:
- moved on the sheet: CAL1, COL_2_TP10, COL_3_TP11, COL_4_TP12, COL_6_TP14, COL_7_TP15, COL_8_TP16, COL_A_TP18, COL_B_TP19, COL_C_TP20, COL_E_TP22, COL_F_TP23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

Commit message: main details roughed out
Parts:
- SWSW_NUMENT1, SW_0_0, SW_3_0, SW_6_0, SW_BACKSL_0, SW_COLON_0, SW_COMMA_0, SW_F11_0, SW_F1_0, SW_F5_0, SW_F9_0, SW_F_0, SW_INS_0, SW_LCTRL_0, SW_LSHIFT_0, SW_NUM0_0, SW_NUM1_0, SW_NUM4_0, SW_NUM7_0, SW_PGUP_0, SW_PRSC_0, SW_TICK_0, SW_V_0, SW_W_0: footprint lib_fp:SW_CAP_IBM_F_ALT -> lib_fp:SW_CAP_IBM_F
- SW_7_0, SW_9_0, SW_BKSP_0, SW_B_0, SW_F10_0, SW_F12_0, SW_HOME_0, SW_I_0, SW_LBRAC_0, SW_LSHIFTX_0, SW_L_0, SW_MINUS_0, SW_NUM0ISOX_0, SW_NUM3_0, SW_NUM8_0, SW_PERIOD_0, SW_RBRAC_0: footprint lib_fp:SW_CAP_IBM_F -> lib_fp:SW_CAP_IBM_F_ALT
- SW_NUM9_0: value CD_R6 -> CE_R7
- SW_NUMASTR_0: value CE_R7 -> CF_R8; footprint lib_fp:SW_CAP_IBM_F_ALT -> lib_fp:SW_CAP_IBM_F
- SW_NUMLK_0: value CC_R6 -> CC_R8
- SW_NUMMIN_0: value CE_R6 -> CF_R7; footprint lib_fp:SW_CAP_IBM_F_ALT -> lib_fp:SW_CAP_IBM_F
- renumbered SW_LSHIFT_1 to SW_1_0, SW_JIS4_0 to SW_JIS3_0, SW_JIS3_0 to SW_JIS4_0
Connections:
- net COL_6: now also SW_JIS3_0.COL; no longer SW_JIS4_0.COL
- net COL_7: now also SW_JIS4_0.COL; no longer SW_JIS3_0.COL
- net COL_9: now also CAL1.COL; no longer SW_RSHIFT_0.COL
- net COL_A: now also SW_RSHIFT_0.COL; no longer CAL1.COL
- net COL_E: no longer SW_NUMMIN_0.COL
- net ROW_1: now also SW_RCTRL_1.ROW; no longer SW_RSHIFT_0.ROW
- net ROW_2: now also SW_RSHIFT_0.ROW; no longer SWSW_NUMENT1.ROW, SW_RCTRL_1.ROW
- net ROW_3: now also SWSW_NUMENT1.ROW
- net ROW_6: no longer SW_NUMMIN_0.ROW
- net ROW_7: now also SW_NUMMIN_0.ROW
Other:
- moved on the sheet: CAL1, SWSW_NUMENT1, SW_JIS3_0, SW_JIS4_0, SW_NUMMIN_0, SW_RCTRL_1, SW_RSHIFT_0

Commit message: save progress
Parts:
- removed H1, H12, H17, H19, H2, H20, H21, H22, H23, H25, H29, H3, H32, H35, H39, H4, H45, H46, H47, H48, H49, H5, H50, H51, H52, H54, H56, H6, H9: HOLE, lib_fp:HOLE, symbol lib_sch:HOLE
- renumbered H7 to H1, H18 to H10, H31 to H11, H27 to H12, H28 to H13, H30 to H14, H26 to H15, H40 to H16, H37 to H17, H36 to H18, H38 to H19, H8 to H2, H33 to H20, H34 to H21, H43 to H22, H44 to H23, H41 to H24, H42 to H25, H55 to H26, H53 to H27, H63 to H28, H59 to H29, H15 to H3, H61 to H30, H60 to H31, H62 to H32, H57 to H33, H58 to H34, H16 to H4, H11 to H5, H13 to H6, H14 to H7, H10 to H8, H24 to H9
Connections:
- net COL_F: now also SW_NUMMIN_0.COL
Other:
- moved on the sheet: COL_1_TP9, COL_2_TP10, COL_3_TP11, COL_4_TP12, COL_5_TP13, COL_6_TP14, COL_7_TP15, COL_8_TP16, COL_9_TP17, COL_A_TP18, COL_B_TP19, COL_C_TP20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
